File: Hardware/915MHz/LoRa_1W_Breakout.sch (EAGLE design)
At the start: 26 parts, among them U4 E19-915M30S

Commit message: Add 433 and 868
Parts:
- removed LOGO1: SFE_LOGO_NAME_FLAME.1_INCH, SparkFun-Aesthetics:SFE_LOGO_NAME_FLAME.1_INCH
- added U$5: SPARKX-LOGO5, SparkX:SPARKX-LOGO5
- C8: value 68uF -> 47uF; device SparkFun-Capacitors:68UF-POLAR-EIA3528-10V-10%(TANT) -> SparkFun-Capacitors:47UF-POLAR-EIA3528-10V-10%
- E1: device SparkFun-RF:ANTENNA-SMA-GROUNDEDEDGE_RPSMA_SMD -> SparkFun-RF:ANTENNA-SMA-GROUNDEDEDGE_RPSMA
Other:
- note added: "Board thickness: 1.6mm"
- note added: "Copper Thickness (1oz): 1.4mil/0.035mm"
- note added: "Dielectric thickness: 1.53mm"
- note added: "Er: 4.5"
- note added: "Microstrip Calculation:"
- note added: "Polygon Isolation: 4mil/0.1016mm"
- note added: "RF Trace Width: 29.1mil/0.74mm"
- note added: "https://chemandy.com/calculators/coplanar-waveguide-with-ground-calculator.htm"
Changed lines of the file:
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@@
 <part name="FD3" library="SparkFun-Aesthetics" deviceset="FIDUCIAL" device="UFIDUCIAL"/>
 <part name="FD4" library="SparkFun-Aesthetics" deviceset="FIDUCIAL" device="UFIDUCIAL"/>
-<part name="LOGO1" library="SparkFun-Aesthetics" deviceset="SFE_LOGO_NAME_FLAME" device=".1_INCH"/>
 <part name="H1" library="SparkFun-Hardware" deviceset="STAND-OFF" device=""/>
 <part name="H2" library="SparkFun-Hardware" deviceset="STAND-OFF" device=""/>
@@
 <part name="GND16" library="SparkFun-PowerSymbols" deviceset="GND" device=""/>
 <part name="GND24" library="SparkFun-PowerSymbols" deviceset="GND" device=""/>
-<part name="VIN_LED" library="SparkFun-Jumpers" deviceset="JUMPER-SMT_2_NC_TRACE" device="_SILK" package3d_urn="urn:adsk.eagle:package:39281/1" value=""/>
+<part name="VIN_LED" library="SparkFun-Jumpers" deviceset="JUMPER-SMT_2_NC_TRACE" device="_SILK" package3d_urn="urn:adsk.eagle:package:39281/1" value="JUMPER-SMT_2_NC_TRACE_SILK"/>
 <part name="D7" library="SparkFun-LED" deviceset="LED-YELLOW" device="0603" value="Yellow"/>
 <part name="GND28" library="SparkFun-PowerSymbols" deviceset="GND" device=""/>
@@
 <part name="R16" library="SparkFun-Resistors" deviceset="100KOHM" device="-0603-1/10W-1%" value="100k"/>
 <part name="SUPPLY12" library="SparkFun-PowerSymbols" deviceset="3.3V" device=""/>
-<part name="E1" library="SparkFun-RF" deviceset="ANTENNA-SMA-GROUNDED" device="EDGE_RPSMA_SMD" value="RP-SMA"/>
+<part name="E1" library="SparkFun-RF" deviceset="ANTENNA-SMA-GROUNDED" device="EDGE_RPSMA" value="RP-SMA"/>
 <part name="GND32" library="SparkFun-PowerSymbols" deviceset="GND" device=""/>
 <part name="R17" library="SparkFun-Resistors" deviceset="100KOHM" device="-0603-1/10W-1%" value="100k"/>
@@
 <part name="R1" library="SparkFun-Resistors" deviceset="1KOHM" device="-0603-1/10W-1%" value="1k"/>
 <part name="FRAME2" library="SparkFun-Aesthetics" deviceset="FRAME-LETTER" device=""/>
-<part name="C8" library="SparkFun-Capacitors" deviceset="68UF-POLAR" device="-EIA3528-10V-10%(TANT)" value="68uF"/>
+<part name="C8" library="SparkFun-Capacitors" deviceset="47UF-POLAR" device="-EIA3528-10V-10%" value="47uF"/>
 <part name="GND17" library="SparkFun-PowerSymbols" deviceset="GND" device=""/>
 <part name="GND1" library="SparkFun-PowerSymbols" deviceset="GND" device=""/>
@@
 <part name="SUPPLY6" library="SparkFun-PowerSymbols" deviceset="5V" device=""/>
 <part name="SUPPLY7" library="SparkFun-PowerSymbols" deviceset="5V" device=""/>
+<part name="U$5" library="SparkX" deviceset="SPARKX-LOGO" device="5" value="SPARKX-LOGO5"/>
 </parts>
 <sheets>
 <sheet>
 <plain>
-<text x="421.894" y="8.636" size="2.54" layer="94">x01</text>
+<text x="241.554" y="8.636" size="2.54" layer="94">x01</text>
 <text x="124.46" y="170.18" size="2.54" layer="94" font="vector" align="center">LoRa Radio 30dBm</text>
+<text x="195.58" y="170.18" size="1.27" layer="97">Board thickness: 1.6mm</text>
+<text x="195.58" y="165.1" size="1.27" layer="97">Er: 4.5</text>
+<text x="195.58" y="172.72" size="1.27" layer="97">Copper Thickness (1oz): 1.4mil/0.035mm</text>
+<text x="195.58" y="160.02" size="1.27" layer="97">RF Trace Width: 29.1mil/0.74mm</text>
+<text x="195.58" y="162.56" size="1.27" layer="97">Polygon Isolation: 4mil/0.1016mm</text>
+<text x="195.58" y="167.64" size="1.27" layer="97">Dielectric thickness: 1.53mm</text>
+<text x="195.58" y="157.48" size="0.762" layer="97">https://chemandy.com/calculators/coplanar-waveguide-with-ground-calculator.htm</text>
+<text x="195.58" y="175.26" size="1.524" layer="97" ratio="15">Microstrip Calculation:</text>
 </plain>
 <instances>
-<instance part="FD1" gate="G$1" x="411.48" y="27.94" smashed="yes"/>
-<instance part="FD2" gate="G$1" x="414.02" y="27.94" smashed="yes"/>
-<instance part="FD3" gate="G$1" x="414.02" y="25.4" smashed="yes"/>
-<instance part="FD4" gate="G$1" x="411.48" y="25.4" smashed="yes"/>
-<instance part="LOGO1" gate="G$1" x="340.36" y="40.64" smashed="yes"/>
-<instance part="H1" gate="G$1" x="419.1" y="27.94" smashed="yes"/>
-<instance part="H2" gate="G$1" x="421.64" y="27.94" smashed="yes"/>
-<instance part="H3" gate="G$1" x="421.64" y="25.4" smashed="yes"/>
-<instance part="H4" gate="G$1" x="419.1" y="25.4" smashed="yes"/>
-<instance part="LOGO3" gate="G$1" x="411.48" y="45.72" smashed="yes"/>
+<instance part="FD1" gate="G$1" x="231.14" y="27.94" smashed="yes"/>
+<instance part="FD2" gate="G$1" x="233.68" y="27.94" smashed="yes"/>
+<instance part="FD3" gate="G$1" x="233.68" y="25.4" smashed="yes"/>
+<instance part="FD4" gate="G$1" x="231.14" y="25.4" smashed="yes"/>
+<instance part="H1" gate="G$1" x="238.76" y="27.94" smashed="yes"/>
+<instance part="H2" gate="G$1" x="241.3" y="27.94" smashed="yes"/>
+<instance part="H3" gate="G$1" x="241.3" y="25.4" smashed="yes"/>
+<instance part="H4" gate="G$1" x="238.76" y="25.4" smashed="yes"/>
+<instance part="LOGO3" gate="G$1" x="236.22" y="45.72" smashed="yes"/>
 <instance part="C5" gate="G$1" x="81.28" y="111.76" smashed="yes">
 <attribute name="NAME" x="82.804" y="114.681" size="1.778" layer="95" font="vector"/>
@@
 <attribute name="VALUE" x="166.624" y="124.46" size="1.778" layer="96" font="vector" rot="R90" align="top-center"/>
 </instance>
-<instance part="GND33" gate="1" x="157.48" y="116.84" smashed="yes">
-<attribute name="VALUE" x="157.48" y="116.586" size="1.778" layer="96" align="top-center"/>
-</instance>
-<instance part="GND34" gate="1" x="165.1" y="116.84" smashed="yes">
-<attribute name="VALUE" x="165.1" y="116.586" size="1.778" layer="96" align="top-center"/>
+<instance part="GND33" gate="1" x="157.48" y="114.3" smashed="yes">
+<attribute name="VALUE" x="157.48" y="114.046" size="1.778" layer="96" align="top-center"/>
+</instance>
+<instance part="GND34" gate="1" x="165.1" y="114.3" smashed="yes">
+<attribute name="VALUE" x="165.1" y="114.046" size="1.778" layer="96" align="top-center"/>
 </instance>
 <instance part="SUPPLY2" gate="G$1" x="101.6" y="119.38" smashed="yes">
@@
 <attribute name="VALUE" x="81.28" y="122.174" size="1.778" layer="96" align="bottom-center"/>
 </instance>
+<instance part="U$5" gate="G$1" x="210.82" y="40.64" smashed="yes"/>
 </instances>
 <busses>
@@
 <pinref part="R18" gate="G$1" pin="1"/>
 <pinref part="GND33" gate="1" pin="GND"/>
+<wire x1="157.48" y1="116.84" x2="157.48" y2="119.38" width="0.1524" layer="91"/>
 </segment>
 <segment>
 <pinref part="R19" gate="G$1" pin="1"/>
 <pinref part="GND34" gate="1" pin="GND"/>
-</segment>
-<segment>
+<wire x1="165.1" y1="116.84" x2="165.1" y2="119.38" width="0.1524" layer="91"/>
+</segment>
+<segment>
