File: Hardware/433MHz/LoRa_1W_Breakout_433MHz.brd (EAGLE design)
At the start: 38.1 x 50.8 mm, 55 parts, among them U4 E19-915M30S

Commit message: Add 433 and 868
Parts:
- removed U$7: (no value), output:915MHZ0
- added U$9: (no value), output:433MHZ0
- U$8: device output:915MHZ0 -> output:433MHZ0
- U4: device SparkFun-RF:E19-915MS1W -> SparkFun-RF:E19-433M30S
- VIN_LED: value (none) -> JUMPER-SMT_2_NC_TRACE_SILK
- moved U$8 19.7 mm to (4.95, 32.8), flipped to the top, turned to 90 degrees
- moved E1 3.25 mm to (28.1, 44.7)
- moved FD2 2.54 mm to (0.64, 47.5)
- moved FD4 2.54 mm to (0.64, 47.5)
- moved H1 2.54 mm to (2.54, 45.7)
- moved H3 2.54 mm to (35.6, 45.7)
- moved U$5 2.54 mm to (12.7, 44.5)
- moved U$69 2.54 mm to (2.54, 38.7)
- moved U$67 2.03 mm to (2.54, 31.0)
- moved U4 1.27 mm to (19.1, 21.6)
- moved U$27 1.27 mm to (5.08, 40.6)
Routing:
- net LORA_!RST!: track 8.71 -> 7.23 mm
- net LORA_D0: track 7.02 -> 5.78 mm
Other:
- board size 38.1 x 50.8 mm -> 38.1 x 48.3 mm

Commit message: Update schematics
Parts:
- U4: value E19-915M30S -> E19-433M30S
- VIN_LED: value JUMPER-SMT_2_NC_TRACE_SILK -> (none)
Changed lines of the file:
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@@
 <layer number="47" name="Measures" color="7" fill="1" visible="no" active="yes"/>
 <layer number="48" name="Document" color="7" fill="1" visible="no" active="yes"/>
-<layer number="49" name="Reference" color="7" fill="1" visible="yes" active="yes"/>
+<layer number="49" name="Reference" color="7" fill="1" visible="no" active="yes"/>
 <layer number="50" name="dxf" color="7" fill="1" visible="no" active="yes"/>
 <layer number="51" name="tDocu" color="6" fill="1" visible="yes" active="yes"/>
@@
 <attribute name="VALUE" x="34.29" y="9.144" size="0.6096" layer="27" font="vector" ratio="20" align="top-center"/>
 </element>
-<element name="VIN_LED" library="SparkFun-Jumpers" package="SMT-JUMPER_2_NC_TRACE_SILK" package3d_urn="urn:adsk.eagle:package:39281/1" value="JUMPER-SMT_2_NC_TRACE_SILK" x="26.67" y="1.27" smashed="yes" rot="MR180">
+<element name="VIN_LED" library="SparkFun-Jumpers" package="SMT-JUMPER_2_NC_TRACE_SILK" package3d_urn="urn:adsk.eagle:package:39281/1" value="" x="26.67" y="1.27" smashed="yes" rot="MR180">
 <attribute name="NAME" x="26.67" y="0.127" size="0.6096" layer="26" font="vector" ratio="20" rot="MR180" align="bottom-center"/>
 <attribute name="VALUE" x="26.67" y="2.413" size="0.6096" layer="28" font="vector" ratio="20" rot="MR180" align="top-center"/>
@@
 <attribute name="VALUE" x="19.05" y="1.905" size="0.6096" layer="27" font="vector" ratio="20" rot="R180" align="top-center"/>
 </element>
-<element name="U4" library="SparkFun-RF" package="E19-433M30S" value="E19-915M30S" x="19.05" y="21.59" smashed="yes" rot="R180">
+<element name="U4" library="SparkFun-RF" package="E19-433M30S" value="E19-433M30S" x="19.05" y="21.59" smashed="yes" rot="R180">
 <attribute name="NAME" x="19.05" y="20.59" size="0.7" layer="25" rot="R180" align="center"/>
 <attribute name="PROD_ID" value="IC-16574" x="19.05" y="21.59" size="1.778" layer="27" font="vector" ratio="15" rot="R180" display="off"/>
