File: Hardware/868MHz/LoRa_1W_Breakout_868MHz.brd (EAGLE design)
At the start: 38.1 x 50.8 mm, 55 parts, among them U4 E19-915M30S

Commit message: Update schematics
Parts:
- U4: value E19-915M30S -> E19-868M30S
- VIN_LED: value JUMPER-SMT_2_NC_TRACE_SILK -> (none)
Changed lines of the file:
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@@
 <attribute name="VALUE" x="34.29" y="9.144" size="0.6096" layer="27" font="vector" ratio="20" align="top-center"/>
 </element>
-<element name="VIN_LED" library="SparkFun-Jumpers" package="SMT-JUMPER_2_NC_TRACE_SILK" package3d_urn="urn:adsk.eagle:package:39281/1" value="JUMPER-SMT_2_NC_TRACE_SILK" x="26.67" y="1.27" smashed="yes" rot="MR180">
+<element name="VIN_LED" library="SparkFun-Jumpers" package="SMT-JUMPER_2_NC_TRACE_SILK" package3d_urn="urn:adsk.eagle:package:39281/1" value="" x="26.67" y="1.27" smashed="yes" rot="MR180">
 <attribute name="NAME" x="26.67" y="0.127" size="0.6096" layer="26" font="vector" ratio="20" rot="MR180" align="bottom-center"/>
 <attribute name="VALUE" x="26.67" y="2.413" size="0.6096" layer="28" font="vector" ratio="20" rot="MR180" align="top-center"/>
@@
 <attribute name="VALUE" x="19.05" y="1.905" size="0.6096" layer="27" font="vector" ratio="20" rot="R180" align="top-center"/>
 </element>
-<element name="U4" library="SparkFun-RF" package="E19-915M30S" value="E19-915M30S" x="19.05" y="22.86" smashed="yes" rot="R180">
+<element name="U4" library="SparkFun-RF" package="E19-915M30S" value="E19-868M30S" x="19.05" y="22.86" smashed="yes" rot="R180">
 <attribute name="NAME" x="19.05" y="21.86" size="0.7" layer="25" rot="R180" align="center"/>
 <attribute name="PROD_ID" value="IC-16573" x="19.05" y="22.86" size="1.778" layer="27" font="vector" ratio="15" rot="R180" display="off"/>
